File: eagle/RPI_Clock.sch (EAGLE design)
At the start: 27 parts, among them T1 IN-12, T2 IN-12, T3 IN-12, T4 IN-12, T5 IN-12, T6 IN-12, U1 K155ID1, U11 74HC595, U2 K155ID1, U3 K155ID1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

Commit message: Updated Eagle design files with 1.3 version
Parts:
- removed ULN2003: ULN2003D1013TR, EE_copy:ULN2003D1013TR
- added U5: ULN2003A, TimeExpander:ULN2003A
- R7, R8, R9: device EE_copy:RESISTOR0805 -> TimeExpander:ANODE_RESISTOR
- renumbered U$1 to U10
Connections:
- net +5V: now also R7.P$2, R8.P$2, R9.P$2; no longer R7.2, R8.2, R9.2
- net GND: now also U5.GND; no longer ULN2003.GND
- net N$47: now also U5.IN1; no longer ULN2003.IN1
- net N$48: now also U5.IN2; no longer ULN2003.IN2
- net N$49: now also R7.P$1, U5.OUT1; no longer R7.1, ULN2003.OUT1
- net N$50: now also R8.P$1, U5.OUT2; no longer R8.1, ULN2003.OUT2
- net N$51: now also R9.P$1, U5.OUT3; no longer R9.1, ULN2003.OUT3
- net N$52: now also U5.IN3; no longer ULN2003.IN3
